File: PCB/LEDs.kicad_sch (KiCad schematic)
At the start: 13 parts

Commit message: schematic done?
Parts:
- renumbered C17 to C18, C18 to C19, C19 to C20, C20 to C21
Changed lines of the file:
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@@
 		(dnp no)
 		(fields_autoplaced yes)
-		(property "Reference" "#PWR053"
+		(property "Reference" "#PWR054"
 			(at 86.36 80.01 0)
 			(effects
@@
 			(project ""
 				(path "/f410b0a0-725c-464e-80be-c0074224226d/7f2ee157-0544-4b4f-a393-7ad097fd1635"
-					(reference "#PWR053")
+					(reference "#PWR054")
 					(unit 1)
 				)
@@
 		(dnp no)
 		(fields_autoplaced yes)
-		(property "Reference" "#PWR055"
+		(property "Reference" "#PWR056"
 			(at 106.68 95.25 0)
 			(effects
@@
 			(project "OTCboard"
 				(path "/f410b0a0-725c-464e-80be-c0074224226d/7f2ee157-0544-4b4f-a393-7ad097fd1635"
-					(reference "#PWR055")
+					(reference "#PWR056")
 					(unit 1)
 				)
@@
 		(dnp no)
 		(fields_autoplaced yes)
-		(property "Reference" "#PWR061"
+		(property "Reference" "#PWR062"
 			(at 154.94 80.01 0)
 			(effects
@@
 			(project "OTCboard"
 				(path "/f410b0a0-725c-464e-80be-c0074224226d/7f2ee157-0544-4b4f-a393-7ad097fd1635"
-					(reference "#PWR061")
+					(reference "#PWR062")
 					(unit 1)
 				)
@@
 		(dnp no)
 		(fields_autoplaced yes)
-		(property "Reference" "#PWR058"
+		(property "Reference" "#PWR059"
 			(at 139.7 87.63 0)
 			(effects
@@
 			(project "OTCboard"
 				(path "/f410b0a0-725c-464e-80be-c0074224226d/7f2ee157-0544-4b4f-a393-7ad097fd1635"
-					(reference "#PWR058")
+					(reference "#PWR059")
 					(unit 1)
 				)
@@
 		(dnp no)
 		(fields_autoplaced yes)
-		(property "Reference" "C20"
+		(property "Reference" "C21"
 			(at 173.99 85.0962 0)
 			(effects
@@
 			(project "OTCboard"
 				(path "/f410b0a0-725c-464e-80be-c0074224226d/7f2ee157-0544-4b4f-a393-7ad097fd1635"
-					(reference "C20")
+					(reference "C21")
 					(unit 1)
 				)
@@
 		(dnp no)
 		(fields_autoplaced yes)
-		(property "Reference" "#PWR057"
+		(property "Reference" "#PWR058"
 			(at 121.92 80.01 0)
 			(effects
@@
 			(project "OTCboard"
 				(path "/f410b0a0-725c-464e-80be-c0074224226d/7f2ee157-0544-4b4f-a393-7ad097fd1635"
-					(reference "#PWR057")
+					(reference "#PWR058")
 					(unit 1)
 				)
@@
 		(dnp no)
 		(fields_autoplaced yes)
-		(property "Reference" "#PWR056"
+		(property "Reference" "#PWR057"
 			(at 121.92 67.31 0)
 			(effects
@@
 			(project "OTCboard"
 				(path "/f410b0a0-725c-464e-80be-c0074224226d/7f2ee157-0544-4b4f-a393-7ad097fd1635"
-					(reference "#PWR056")
+					(reference "#PWR057")
 					(unit 1)
 				)
@@
 		(dnp no)
 		(fields_autoplaced yes)
-		(property "Reference" "#PWR060"
+		(property "Reference" "#PWR061"
 			(at 154.94 67.31 0)
 			(effects
@@
 			(project "OTCboard"
 				(path "/f410b0a0-725c-464e-80be-c0074224226d/7f2ee157-0544-4b4f-a393-7ad097fd1635"
-					(reference "#PWR060")
+					(reference "#PWR061")
 					(unit 1)
 				)
@@
 		(dnp no)
 		(fields_autoplaced yes)
-		(property "Reference" "#PWR064"
+		(property "Reference" "#PWR065"
 			(at 190.5 67.31 0)
 			(effects
@@
 			(project "OTCboard"
 				(path "/f410b0a0-725c-464e-80be-c0074224226d/7f2ee157-0544-4b4f-a393-7ad097fd1635"
-					(reference "#PWR064")
+					(reference "#PWR065")
 					(unit 1)
 				)
@@
 		(dnp no)
 		(fields_autoplaced yes)
-		(property "Reference" "#PWR054"
+		(property "Reference" "#PWR055"
 			(at 106.68 87.63 0)
 			(effects
@@
 			(project "OTCboard"
 				(path "/f410b0a0-725c-464e-80be-c0074224226d/7f2ee157-0544-4b4f-a393-7ad097fd1635"
-					(reference "#PWR054")
+					(reference "#PWR055")
 					(unit 1)
 				)
@@
 		(dnp no)
 		(fields_autoplaced yes)
-		(property "Reference" "C18"
+		(property "Reference" "C19"
 			(at 109.22 85.0962 0)
 			(effects
@@
 			(project "OTCboard"
 				(path "/f410b0a0-725c-464e-80be-c0074224226d/7f2ee157-0544-4b4f-a393-7ad097fd1635"
-					(reference "C18")
+					(reference "C19")
 					(unit 1)
 				)
@@
 		(dnp no)
 		(fields_autoplaced yes)
-		(property "Reference" "#PWR050"
+		(property "Reference" "#PWR051"
 			(at 73.66 87.63 0)
 			(effects
@@
 			(project "OTCboard"
 				(path "/f410b0a0-725c-464e-80be-c0074224226d/7f2ee157-0544-4b4f-a393-7ad097fd1635"
-					(reference "#PWR050")
+					(reference "#PWR051")
 					(unit 1)
 				)
@@
 		(dnp no)
 		(fields_autoplaced yes)
-		(property "Reference" "#PWR063"
+		(property "Reference" "#PWR064"
 			(at 171.45 95.25 0)
 			(effects
@@
 			(project "OTCboard"
 				(path "/f410b0a0-725c-464e-80be-c0074224226d/7f2ee157-0544-4b4f-a393-7ad097fd1635"
-					(reference "#PWR063")
+					(reference "#PWR064")
 					(unit 1)
 				)
@@
 		(dnp no)
 		(fields_autoplaced yes)
-		(property "Reference" "#PWR065"
+		(property "Reference" "#PWR066"
 			(at 194.31 80.01 0)
 			(effects
@@
 			(project "OTCboard"
 				(path "/f410b0a0-725c-464e-80be-c0074224226d/7f2ee157-0544-4b4f-a393-7ad097fd1635"
-					(reference "#PWR065")
+					(reference "#PWR066")
 					(unit 1)
 				)
@@
 		(dnp no)
 		(fields_autoplaced yes)
-		(property "Reference" "C19"
+		(property "Reference" "C20"
 			(at 142.24 85.0962 0)
 			(effects
@@
 			(project "OTCboard"
 				(path "/f410b0a0-725c-464e-80be-c0074224226d/7f2ee157-0544-4b4f-a393-7ad097fd1635"
-					(reference "C19")
+					(reference "C20")
 					(unit 1)
 				)
@@
 		(dnp no)
 		(fields_autoplaced yes)
-		(property "Reference" "#PWR051"
+		(property "Reference" "#PWR052"
 			(at 73.66 95.25 0)
 			(effects
@@
 			(project "OTCboard"
 				(path "/f410b0a0-725c-464e-80be-c0074224226d/7f2ee157-0544-4b4f-a393-7ad097fd1635"
-					(reference "#PWR051")
+					(reference "#PWR052")
 					(unit 1)
 				)
@@
 		(dnp no)
 		(fields_autoplaced yes)
-		(property "Reference" "#PWR062"
+		(property "Reference" "#PWR063"
 			(at 171.45 87.63 0)
 			(effects
@@
 			(project "OTCboard"
 				(path "/f410b0a0-725c-464e-80be-c0074224226d/7f2ee157-0544-4b4f-a393-7ad097fd1635"
-					(reference "#PWR062")
+					(reference "#PWR063")
 					(unit 1)
 				)
@@
 		(dnp no)
 		(fields_autoplaced yes)
-		(property "Reference" "#PWR052"
+		(property "Reference" "#PWR053"
 			(at 86.36 67.31 0)
 			(effects
@@
 			(project ""
 				(path "/f410b0a0-725c-464e-80be-c0074224226d/7f2ee157-0544-4b4f-a393-7ad097fd1635"
-					(reference "#PWR052")
+					(reference "#PWR053")
 					(unit 1)
 				)
@@
 		(dnp no)
 		(fields_autoplaced yes)
-		(property "Reference" "C17"
+		(property "Reference" "C18"
 			(at 76.2 85.0962 0)
 			(effects
@@
 			(project ""
 				(path "/f410b0a0-725c-464e-80be-c0074224226d/7f2ee157-0544-4b4f-a393-7ad097fd1635"
-					(reference "C17")
+					(reference "C18")
 					(unit 1)
 				)
@@
 		(dnp no)
 		(fields_autoplaced yes)
-		(property "Reference" "#PWR059"
+		(property "Reference" "#PWR060"
 			(at 139.7 95.25 0)
 			(effects
@@
 			(project "OTCboard"
 				(path "/f410b0a0-725c-464e-80be-c0074224226d/7f2ee157-0544-4b4f-a393-7ad097fd1635"
-					(reference "#PWR059")
-					(unit 1)
-				)
+					(reference "#PWR060")
+					(unit 1)
+				)

Commit message: analog signal design research
Parts:
- renumbered C18 to C22, C19 to C23, C20 to C24, C21 to C25, R7 to R11
Changed lines of the file:
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@@
 		(dnp no)
 		(fields_autoplaced yes)
-		(property "Reference" "#PWR054"
+		(property "Reference" "#PWR058"
 			(at 86.36 80.01 0)
 			(effects
@@
 			(project ""
 				(path "/f410b0a0-725c-464e-80be-c0074224226d/7f2ee157-0544-4b4f-a393-7ad097fd1635"
-					(reference "#PWR054")
+					(reference "#PWR058")
 					(unit 1)
 				)
@@
 		(dnp no)
 		(fields_autoplaced yes)
-		(property "Reference" "#PWR056"
+		(property "Reference" "#PWR060"
 			(at 106.68 95.25 0)
 			(effects
@@
 			(project "OTCboard"
 				(path "/f410b0a0-725c-464e-80be-c0074224226d/7f2ee157-0544-4b4f-a393-7ad097fd1635"
-					(reference "#PWR056")
+					(reference "#PWR060")
 					(unit 1)
 				)
@@
 		(dnp no)
 		(fields_autoplaced yes)
-		(property "Reference" "#PWR062"
+		(property "Reference" "#PWR066"
 			(at 154.94 80.01 0)
 			(effects
@@
 			(project "OTCboard"
 				(path "/f410b0a0-725c-464e-80be-c0074224226d/7f2ee157-0544-4b4f-a393-7ad097fd1635"
-					(reference "#PWR062")
+					(reference "#PWR066")
 					(unit 1)
 				)
@@
 		(dnp no)
 		(fields_autoplaced yes)
-		(property "Reference" "#PWR059"
+		(property "Reference" "#PWR063"
 			(at 139.7 87.63 0)
 			(effects
@@
 			(project "OTCboard"
 				(path "/f410b0a0-725c-464e-80be-c0074224226d/7f2ee157-0544-4b4f-a393-7ad097fd1635"
-					(reference "#PWR059")
+					(reference "#PWR063")
 					(unit 1)
 				)
@@
 		(dnp no)
 		(fields_autoplaced yes)
-		(property "Reference" "C21"
+		(property "Reference" "C25"
 			(at 173.99 85.0962 0)
 			(effects
@@
 			(project "OTCboard"
 				(path "/f410b0a0-725c-464e-80be-c0074224226d/7f2ee157-0544-4b4f-a393-7ad097fd1635"
-					(reference "C21")
+					(reference "C25")
 					(unit 1)
 				)
@@
 		(dnp no)
 		(fields_autoplaced yes)
-		(property "Reference" "#PWR058"
+		(property "Reference" "#PWR062"
 			(at 121.92 80.01 0)
 			(effects
@@
 			(project "OTCboard"
 				(path "/f410b0a0-725c-464e-80be-c0074224226d/7f2ee157-0544-4b4f-a393-7ad097fd1635"
-					(reference "#PWR058")
+					(reference "#PWR062")
 					(unit 1)
 				)
@@
 		(dnp no)
 		(fields_autoplaced yes)
-		(property "Reference" "#PWR057"
+		(property "Reference" "#PWR061"
 			(at 121.92 67.31 0)
 			(effects
@@
 			(project "OTCboard"
 				(path "/f410b0a0-725c-464e-80be-c0074224226d/7f2ee157-0544-4b4f-a393-7ad097fd1635"
-					(reference "#PWR057")
+					(reference "#PWR061")
 					(unit 1)
 				)
@@
 		(dnp no)
 		(fields_autoplaced yes)
-		(property "Reference" "#PWR061"
+		(property "Reference" "#PWR065"
 			(at 154.94 67.31 0)
 			(effects
@@
 			(project "OTCboard"
 				(path "/f410b0a0-725c-464e-80be-c0074224226d/7f2ee157-0544-4b4f-a393-7ad097fd1635"
-					(reference "#PWR061")
+					(reference "#PWR065")
 					(unit 1)
 				)
@@
 		(dnp no)
 		(fields_autoplaced yes)
-		(property "Reference" "#PWR065"
+		(property "Reference" "#PWR069"
 			(at 190.5 67.31 0)
 			(effects
@@
 			(project "OTCboard"
 				(path "/f410b0a0-725c-464e-80be-c0074224226d/7f2ee157-0544-4b4f-a393-7ad097fd1635"
-					(reference "#PWR065")
+					(reference "#PWR069")
 					(unit 1)
 				)
@@
 		(dnp no)
 		(fields_autoplaced yes)
-		(property "Reference" "#PWR055"
+		(property "Reference" "#PWR059"
 			(at 106.68 87.63 0)
 			(effects
@@
 			(project "OTCboard"
 				(path "/f410b0a0-725c-464e-80be-c0074224226d/7f2ee157-0544-4b4f-a393-7ad097fd1635"
-					(reference "#PWR055")
+					(reference "#PWR059")
 					(unit 1)
 				)
@@
 		(dnp no)
 		(fields_autoplaced yes)
-		(property "Reference" "C19"
+		(property "Reference" "C23"
 			(at 109.22 85.0962 0)
 			(effects
@@
 			(project "OTCboard"
 				(path "/f410b0a0-725c-464e-80be-c0074224226d/7f2ee157-0544-4b4f-a393-7ad097fd1635"
-					(reference "C19")
+					(reference "C23")
 					(unit 1)
 				)
@@
 		(dnp no)
 		(fields_autoplaced yes)
-		(property "Reference" "#PWR051"
+		(property "Reference" "#PWR055"
 			(at 73.66 87.63 0)
 			(effects
@@
 			(project "OTCboard"
 				(path "/f410b0a0-725c-464e-80be-c0074224226d/7f2ee157-0544-4b4f-a393-7ad097fd1635"
-					(reference "#PWR051")
+					(reference "#PWR055")
 					(unit 1)
 				)
@@
 		(dnp no)
 		(fields_autoplaced yes)
-		(property "Reference" "#PWR064"
+		(property "Reference" "#PWR068"
 			(at 171.45 95.25 0)
 			(effects
@@
 			(project "OTCboard"
 				(path "/f410b0a0-725c-464e-80be-c0074224226d/7f2ee157-0544-4b4f-a393-7ad097fd1635"
-					(reference "#PWR064")
+					(reference "#PWR068")
 					(unit 1)
 				)
@@
 		(dnp no)
 		(fields_autoplaced yes)
-		(property "Reference" "#PWR066"
+		(property "Reference" "#PWR070"
 			(at 194.31 80.01 0)
 			(effects
@@
 			(project "OTCboard"
 				(path "/f410b0a0-725c-464e-80be-c0074224226d/7f2ee157-0544-4b4f-a393-7ad097fd1635"
-					(reference "#PWR066")
+					(reference "#PWR070")
 					(unit 1)
 				)
@@
 		(dnp no)
 		(fields_autoplaced yes)
-		(property "Reference" "R7"
+		(property "Reference" "R11"
 			(at 196.215 69.8499 0)
 			(effects
@@
 			(project ""
 				(path "/f410b0a0-725c-464e-80be-c0074224226d/7f2ee157-0544-4b4f-a393-7ad097fd1635"
-					(reference "R7")
+					(reference "R11")
 					(unit 1)
 				)
@@
 		(dnp no)
 		(fields_autoplaced yes)
-		(property "Reference" "C20"
+		(property "Reference" "C24"
 			(at 142.24 85.0962 0)
 			(effects
@@
 			(project "OTCboard"
 				(path "/f410b0a0-725c-464e-80be-c0074224226d/7f2ee157-0544-4b4f-a393-7ad097fd1635"
-					(reference "C20")
+					(reference "C24")
 					(unit 1)
 				)
@@
 		(dnp no)
 		(fields_autoplaced yes)
-		(property "Reference" "#PWR052"
+		(property "Reference" "#PWR056"
 			(at 73.66 95.25 0)
 			(effects
@@
 			(project "OTCboard"
 				(path "/f410b0a0-725c-464e-80be-c0074224226d/7f2ee157-0544-4b4f-a393-7ad097fd1635"
-					(reference "#PWR052")
+					(reference "#PWR056")
 					(unit 1)
 				)
@@
 		(dnp no)
 		(fields_autoplaced yes)
-		(property "Reference" "#PWR063"
+		(property "Reference" "#PWR067"
 			(at 171.45 87.63 0)
 			(effects
@@
 			(project "OTCboard"
 				(path "/f410b0a0-725c-464e-80be-c0074224226d/7f2ee157-0544-4b4f-a393-7ad097fd1635"
-					(reference "#PWR063")
+					(reference "#PWR067")
 					(unit 1)
 				)
@@
 		(dnp no)
 		(fields_autoplaced yes)
-		(property "Reference" "#PWR053"
+		(property "Reference" "#PWR057"
 			(at 86.36 67.31 0)
 			(effects
@@
 			(project ""
 				(path "/f410b0a0-725c-464e-80be-c0074224226d/7f2ee157-0544-4b4f-a393-7ad097fd1635"
-					(reference "#PWR053")
+					(reference "#PWR057")
 					(unit 1)
 				)
@@
 		(dnp no)
 		(fields_autoplaced yes)
-		(property "Reference" "C18"
+		(property "Reference" "C22"
 			(at 76.2 85.0962 0)
 			(effects
@@
 			(project ""
 				(path "/f410b0a0-725c-464e-80be-c0074224226d/7f2ee157-0544-4b4f-a393-7ad097fd1635"
-					(reference "C18")
+					(reference "C22")
 					(unit 1)
 				)
@@
 		(dnp no)
 		(fields_autoplaced yes)
-		(property "Reference" "#PWR060"
+		(property "Reference" "#PWR064"
 			(at 139.7 95.25 0)
 			(effects
@@
 			(project "OTCboard"
 				(path "/f410b0a0-725c-464e-80be-c0074224226d/7f2ee157-0544-4b4f-a393-7ad097fd1635"
-					(reference "#PWR060")
-					(unit 1)
-				)
+					(reference "#PWR064")
+					(unit 1)
+				)
