File: PCB/OTCboard.kicad_pcb (KiCad board)
At the start: 2 copper layers, 60 x 60 mm, 59 parts, among them J1 USB_C_Receptacle_USB2.0_16P, U1 STM32G431CBTx, U2 MCP1826S, U3 DRV5055A3xDBZxQ1, U4 DRV5055A3xDBZxQ1, U5 DRV5055A3xDBZxQ1, U6 DRV5055A3xDBZxQ1, Y1 Crystal

Commit message: schematic done?
Parts:
- added C21: 0.1u, Capacitor_SMD:C_0603_1608Metric_Pad1.08x0.95mm_HandSolder, F.Cu at (91.5, 83.1)
- added S1: TL3365AF180QG, Reset Button:TL3365AF180QG, F.Cu at (111.8, 54.2)
- added SW1: SW_SPDT, Slide Switch:CLSB12B01T, F.Cu at (119.5, 54.1)
- C1, C2: value 26p -> 16p
- C10: value 10u -> 0.1uF; footprint Capacitor_SMD:C_0805_2012Metric_Pad1.18x1.45mm_HandSolder -> Capacitor_SMD:C_0603_1608Metric_Pad1.08x0.95mm_HandSolder
- C13: value 0.1u -> 10u; footprint Capacitor_SMD:C_0603_1608Metric_Pad1.08x0.95mm_HandSolder -> Capacitor_SMD:C_0805_2012Metric_Pad1.18x1.45mm_HandSolder
- C3: value 0.1u -> 100n
- C4: value 4.7uF -> 0.1u; footprint Capacitor_SMD:C_0805_2012Metric_Pad1.18x1.45mm_HandSolder -> Capacitor_SMD:C_0603_1608Metric_Pad1.08x0.95mm_HandSolder
- C5: value 0.1uF -> 4.7uF; footprint Capacitor_SMD:C_0603_1608Metric_Pad1.08x0.95mm_HandSolder -> Capacitor_SMD:C_0805_2012Metric_Pad1.18x1.45mm_HandSolder
- D3, D4, R5, R6, U10, U8: moved to B.Cu
- Y1: value Crystal -> 8M
- moved TP5 73.2 mm to (153.0, 102.0)
- moved TP4 64.0 mm to (134.0, 102.0)
- moved D8 49.0 mm to (130.0, 73.9)
- moved TP6 42.6 mm to (134.0, 83.0)
- moved U6 39.4 mm to (130.0, 79.0)
- moved C3 37.7 mm to (148.1, 69.0), turned to 0 degrees
- moved FB1 34.9 mm to (81.8, 66.2)
- moved C9 34.8 mm to (85.3, 67.8)
- moved C8 34.7 mm to (85.3, 66.2)
- moved C10 34.7 mm to (85.3, 69.4)
- moved FB2 34.7 mm to (88.9, 67.8)
- moved C6 34.7 mm to (88.9, 66.2)
- moved R2 29.9 mm to (88.1, 58.8)
- moved D4 8.95 mm to (143.8, 53.5), turned to -90 degrees
- moved TP3 7.80 mm to (115.0, 102.0)
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Connections:
- C10 pad 1: +5V -> +3V3A
- C10 pad 2: GND -> GNDA
- C12 pad 1: +3.3V -> +5V
- C17 pad 1: +5V -> +3.3V
- C3 pad 1: /MCU/NRST -> Net-(U1-VBAT)
- C3 pad 2: GND -> +3.3V
- C4 pad 1: +3.3V -> /MCU/NRST
- C7 pad 1: +3V3A -> +3.3V
- C7 pad 2: GNDA -> GND
- U1 pad 1: +3.3V -> Net-(U1-VBAT)
Routing:
- net /USB/USB_D-: track 0.00 -> 16.5 mm
- net /USB/USB_D+: track 0.00 -> 15.7 mm
- removed copper zone on F.Cu, net +3V3A
- removed copper zone on F.Cu, net GNDA
Other:
- board text added: "10 BOOT"

Commit message: analog signal design research
Parts:
- added C22: 0.1u, Capacitor_SMD:C_0603_1608Metric_Pad1.08x0.95mm_HandSolder, F.Cu at (113.0, 90.0)
- added C23: 0.1u, Capacitor_SMD:C_0603_1608Metric_Pad1.08x0.95mm_HandSolder, F.Cu at (132.0, 90.0)
- added C24: 0.1u, Capacitor_SMD:C_0603_1608Metric_Pad1.08x0.95mm_HandSolder, F.Cu at (151.0, 90.0)
- added C25: 0.1u, Capacitor_SMD:C_0603_1608Metric_Pad1.08x0.95mm_HandSolder, F.Cu at (132.0, 71.0)
- added R10: 1k, Resistor_SMD:R_0603_1608Metric_Pad0.98x0.95mm_HandSolder, F.Cu at (130.0, 82.8)
- added R11: 10k, Resistor_SMD:R_0603_1608Metric_Pad0.98x0.95mm_HandSolder, F.Cu at (139.0, 75.6)
- added R8: 1k, Resistor_SMD:R_0603_1608Metric_Pad0.98x0.95mm_HandSolder, F.Cu at (130.0, 101.8)
- added R9: 1k, Resistor_SMD:R_0603_1608Metric_Pad0.98x0.95mm_HandSolder, F.Cu at (149.0, 101.8)
- R3, R4: moved to F.Cu
- R7: value 10k -> 1k
- moved C19 70.8 mm to (150.7, 101.8), turned to 90 degrees
- moved C17 68.1 mm to (112.7, 101.8), turned to -90 degrees
- moved C18 66.7 mm to (131.7, 101.8), turned to -90 degrees
- moved C13 45.6 mm to (139.9, 67.4)
- moved C20 42.6 mm to (128.3, 82.8), turned to -90 degrees
- moved R7 41.1 mm to (111.0, 101.8), turned to -90 degrees
- moved C21 40.2 mm to (131.7, 82.8), turned to 90 degrees
- moved C3 38.2 mm to (111.0, 59.8), turned to 90 degrees
- moved C10 31.3 mm to (116.1, 75.2)
- moved C8 31.3 mm to (116.1, 72.0)
- moved C9 31.3 mm to (116.1, 73.6)
- moved FB1 31.3 mm to (112.6, 72.0)
- moved C6 31.3 mm to (119.7, 72.0), turned to 0 degrees
- moved FB2 31.3 mm to (119.7, 73.6)
- moved R2 28.9 mm to (117.0, 59.6), turned to 0 degrees
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Connections:
- C10 pad 1: +3V3A -> +3.3VA
- C14 pad 1: +3.3V -> +3.3VA
- C15 pad 1: +3.3V -> +3.3VA
- C16 pad 1: +3.3V -> +3.3VA
- C17 pad 1: +3.3V -> /Keys/KEY1
- C18 pad 1: +5V -> /Keys/KEY2
- C19 pad 1: +5V -> /Keys/KEY3
- C20 pad 1: +5V -> +3.3VA
- C21 pad 1: +5V -> /Keys/KEY4
- C8 pad 1: +3V3A -> +3.3VA
- C9 pad 1: +3V3A -> +3.3VA
- FB2 pad 2: +3V3A -> +3.3VA
- R7 pad 1: Net-(D8-DOUT) -> Net-(U4-OUT)
- R7 pad 2: GND -> /Keys/KEY1
- U1 pad 21: +3V3A -> +3.3VA
- U3 pad 1: +3.3V -> +3.3VA
- U3 pad 2: /Keys/KEY1 -> Net-(U3-OUT)
- U3 pad 3: GND -> GNDA
- U4 pad 1: +3.3V -> +3.3VA
- U4 pad 2: /Keys/KEY2 -> Net-(U4-OUT)
- U4 pad 3: GND -> GNDA
- U5 pad 1: +3.3V -> +3.3VA
- U5 pad 2: /Keys/KEY3 -> Net-(U5-OUT)
- U5 pad 3: GND -> GNDA
- U6 pad 1: +3.3V -> +3.3VA
- U6 pad 2: /Keys/KEY4 -> Net-(U6-OUT)
- U6 pad 3: GND -> GNDA
Routing:
- net +5V: track 0.00 -> 85.0 mm, vias 0 -> 5
- net /MCU/NRST: track 0.00 -> 21.5 mm, vias 0 -> 2
- net /USB/VBUSB: track 0.00 -> 10.7 mm
- net Net-(U1-PF1): track 0.00 -> 9.26 mm
- net Net-(U1-PF0): track 0.00 -> 9.25 mm
- net +3.3V: track 0.00 -> 8.81 mm, vias 0 -> 1
- net Net-(SW1-B): track 0.00 -> 3.31 mm
- net /MCU/BOOT: track 0.00 -> 3.16 mm
- net /USB/USB_D+: track 15.7 -> 18.8 mm
- net /USB/USB_D-: track 16.5 -> 19.5 mm
- net /USB/CC2: track 0.00 -> 2.98 mm
- net Net-(U1-VBAT): track 0.00 -> 2.75 mm
- net /USB/CC1: track 0.00 -> 2.65 mm
- net GND: track 0.00 -> 1.70 mm, vias 0 -> 5
- net GNDA: vias 0 -> 1
- added copper zone on B.Cu, net +3.3V
- added copper zone on F.Cu, net +3.3V
- added copper zone on In1.Cu, net +3.3V
- added copper zone on F.Cu, net +3V3A
- added copper zone on F.Cu, net +5V
- added copper zone on F.Cu, net /USB/VBUSB
- added copper zone on In2.Cu, net GND
- added copper zone on F.Cu, net GNDA
- removed copper zone on B.Cu, net GND
Other:
- copper layers 2 -> 4
- board text added: "A"
- board text added: "BOOT 10"
- board text added: "D"
- board text added: "S"
- board text added: "W"
- board text removed: "10 BOOT"

Commit message: routing
Parts:
- removed FB1: FerriteBead, Inductor_SMD:L_0603_1608Metric_Pad1.05x0.95mm_HandSolder
- S1, SW1: moved to B.Cu
- moved U3 38.0 mm to (149.0, 98.1)
- moved U4 19.0 mm to (111.0, 98.0)
- moved U5 19.0 mm to (130.0, 98.0)
- moved R11 4.31 mm to (134.7, 75.6)
- turned C19 to -90 degrees
- turned C21 to -90 degrees
- turned R8 to -90 degrees
- turned S1 to -90 degrees
- turned SW1 to 0 degrees
Connections:
- C10 pad 2: GNDA -> GND
- C8 pad 2: GNDA -> GND
- C9 pad 2: GNDA -> GND
- U1 pad 12: unconnected-(U1-PA4-Pad12) -> /LEDs/AddressableLEDs
- U1 pad 19: GNDA -> GND
- U1 pad 20: +3V3A -> +3.3VA
- U1 pad 25: /LEDs/AddressableLEDs -> unconnected-(U1-PB11-Pad25)
- U3 pad 3: GNDA -> GND
- U4 pad 3: GNDA -> GND
- U5 pad 3: GNDA -> GND
- U6 pad 3: GNDA -> GND
Routing:
- net /Keys/KEY3: track 0.00 -> 67.5 mm
- net +5V: track 85.0 -> 22.6 mm
- net /Keys/KEY2: track 0.00 -> 48.5 mm
- net /Keys/KEY1: track 0.00 -> 45.4 mm
- net GND: track 1.70 -> 44.8 mm, vias 5 -> 83
- net Net-(D7-DOUT): track 0.00 -> 41.9 mm, vias 0 -> 2
- net /Keys/KEY4: track 0.00 -> 30.4 mm
- net /LEDs/AddressableLEDs: track 0.00 -> 24.2 mm, vias 0 -> 2
- net +3.3VA: track 0.00 -> 15.3 mm, vias 0 -> 8
- net Net-(D6-DOUT): track 0.00 -> 14.2 mm, vias 0 -> 2
- net Net-(D5-DOUT): track 0.00 -> 13.2 mm, vias 0 -> 2
- net +3.3V: track 8.81 -> 18.3 mm, vias 1 -> 9
- net Net-(U4-OUT): track 0.00 -> 2.34 mm
- net Net-(U6-OUT): track 0.00 -> 2.34 mm
- net Net-(U5-OUT): track 0.00 -> 2.34 mm
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- added copper zone on In2.Cu, net +3.3V
- added copper zone on F.Cu, net +3.3VA
- added copper zone on In2.Cu, net +3.3VA
- added copper zone on In2.Cu, net +5V
- added copper zone on B.Cu, net GND
- added copper zone on In1.Cu, net GND
- removed copper zone on B.Cu, net +3.3V
- removed copper zone on In1.Cu, net +3.3V
- removed copper zone on F.Cu, net +3V3A
- removed copper zone on F.Cu, net GNDA
