File: PCB/OTCboard.kicad_pcb (KiCad board)
At the start: 4 copper layers, 60 x 60 mm, 69 parts, among them J1 USB_C_Receptacle_USB2.0_16P, SW1 SW_SPDT, U1 STM32G431CBTx, U2 MCP1826S, U3 DRV5055A3xDBZxQ1, U4 DRV5055A3xDBZxQ1, U5 DRV5055A3xDBZxQ1, U6 DRV5055A3xDBZxQ1, Y1 8M

Commit message: gerbers and added to cart on jlc
Parts:
- added G***: LOGO, LOGO, B.Cu at (150.0, 71.0)
- moved H3 7.40 mm to (155.0, 85.0)
- moved TP2 4.80 mm to (149.2, 53.0)
- moved TP1 4.70 mm to (149.2, 57.8)
- moved H4 4.39 mm to (105.0, 85.0)
Routing:
- net GND: track 44.8 -> 9.49 mm, vias 83 -> 126
- net +5V: track 22.6 -> 11.9 mm, vias 5 -> 8
- net +3.3V: track 18.3 -> 20.3 mm
- net Net-(D7-DOUT): track 41.9 -> 41.2 mm
Other:
- board text added: "01"
- board text added: "727"
- board text added: "BOOT"
- board text added: "RESET"
- board text removed: "BOOT 10"
